File: WS2811 Expander.kicad_pcb (KiCad board)
At the start: 2 copper layers, 33.7 x 27 mm, 28 parts, among them J1  , J2  , J3 , Q1  MMBT3904, Q2 IRLR7821PBF, Q3  MMBT3904, Q4  MMBT3904, Q5 IRLR7821PBF, Q6 IRLR7821PBF, U1 WS2811

Commit message: updated design, new test app, ready for assembly
Parts:
- removed  : , Pin_Headers:Pin_Header_Straight_1x01_Pitch2.54mm (x3)
- added REF**: Via-0.6mm, Via-0.6mm, F.Cu at (161.0, 43.9)
- added REF**: Via-0.6mm, Via-0.6mm, F.Cu at (161.2, 36.0)
- added REF**: Via-0.6mm, Via-0.6mm, F.Cu at (161.7, 35.5)
- added REF**: Via-0.6mm, Via-0.6mm, F.Cu at (162.2, 36.5)
- added REF**: Via-0.6mm, Via-0.6mm, F.Cu at (162.2, 36.0)
- added REF**: Via-0.6mm, Via-0.6mm, F.Cu at (161.2, 36.5)
- added REF**: Via-0.6mm, Via-0.6mm, F.Cu at (162.2, 35.5)
- added REF**: Via-0.6mm, Via-0.6mm, F.Cu at (161.7, 36.5)
- added REF**: Via-0.6mm, Via-0.6mm, F.Cu at (161.7, 36.0)
- added REF**: Via-0.6mm, Via-0.6mm, F.Cu at (161.2, 35.5)
- added REF**: Via-0.6mm, Via-0.6mm, F.Cu at (162.2, 29.3)
- added REF**: Via-0.6mm, Via-0.6mm, F.Cu at (161.5, 43.4)
- added REF**: Via-0.6mm, Via-0.6mm, F.Cu at (161.7, 29.3)
- added REF**: Via-0.6mm, Via-0.6mm, F.Cu at (161.2, 29.3)
- added REF**: Via-0.6mm, Via-0.6mm, F.Cu at (162.2, 28.8)
- added REF**: Via-0.6mm, Via-0.6mm, F.Cu at (161.7, 28.8)
- added REF**: Via-0.6mm, Via-0.6mm, F.Cu at (161.2, 28.8)
- added REF**: Via-0.6mm, Via-0.6mm, F.Cu at (162.2, 28.3)
- added REF**: Via-0.6mm, Via-0.6mm, F.Cu at (161.7, 28.3)
- added REF**: Via-0.6mm, Via-0.6mm, F.Cu at (161.2, 28.3)
- added REF**: Via-0.6mm, Via-0.6mm, F.Cu at (162.0, 42.9)
- added REF**: Via-0.6mm, Via-0.6mm, F.Cu at (162.0, 43.4)
- added REF**: Via-0.6mm, Via-0.6mm, F.Cu at (161.5, 43.9)
- added REF**: Via-0.6mm, Via-0.6mm, F.Cu at (161.0, 43.4)
- added REF**: Via-0.6mm, Via-0.6mm, F.Cu at (161.5, 42.9)
- added REF**: Via-0.6mm, Via-0.6mm, F.Cu at (161.0, 42.9)
- added REF**: Via-0.6mm, Via-0.6mm, F.Cu at (162.0, 43.9)
- C1 : footprint Capacitors_SMD:C_0805 -> Capacitors_SMD:C_0603
- R1, R12, R13, R14, R2, R3: footprint Resistors_SMD:R_0805 -> Resistors_SMD:R_0603
- R11 : renamed from  ; footprint Resistors_SMD:R_0805 -> Resistors_SMD:R_0603
- R4 : footprint Resistors_SMD:R_0805 -> Resistors_SMD:R_0603
- R5 : footprint Resistors_SMD:R_0805 -> Resistors_SMD:R_0603
- R6 : footprint Resistors_SMD:R_0805 -> Resistors_SMD:R_0603
- R7 : renamed from  ; footprint Resistors_SMD:R_0805 -> Resistors_SMD:R_0603
- R8 : renamed from  ; footprint Resistors_SMD:R_0805 -> Resistors_SMD:R_0603
Other:
- board text added: "EagleDecorations WS2811 Expander V1.1 Automated"
- board text removed: "EagleDecorations WS2811 Expander V1.0"
- board text removed: "Fill"
