File: WS2811 Expander.sch (KiCad schematic (older format))
At the start: 28 parts, among them J1 , J2 , J3 , J5 , J6 , J7 , Q1 MMBT3904, Q2 IRLR7821PBF, Q3 MMBT3904, Q4 MMBT3904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

Commit message: updated design, new test app, ready for assembly
Parts:
- C1: footprint Capacitors_SMD:C_0805 -> Capacitors_SMD:C_0603; LCSC (none) -> C14663
- Q1, Q3, Q4: LCSC (none) -> C20526
- Q2, Q5, Q6: value IRLR7821PBF -> AOD4184A; footprint TO_SOT_Packages_SMD:TO-252-3_TabPin4 -> TO_SOT_Packages_SMD:TO-252-2; LCSC (none) -> C99124
- R1, R2, R3, R4, R5, R6: footprint Resistors_SMD:R_0805 -> Resistors_SMD:R_0603; LCSC (none) -> C21190
- R11: LCSC (none) -> C23140
- R12, R13, R14: footprint Resistors_SMD:R_0805 -> Resistors_SMD:R_0603; LCSC (none) -> C25804
- R7: LCSC (none) -> C22775
- R8: LCSC (none) -> C13167
- U1: LCSC (none) -> C114581
Changed lines of the file:
@@
 F 2 "TO_SOT_Packages_SMD:SOT-23" H 5050 2875 50  0001 L CIN
 F 3 "https://www.fairchildsemi.com/datasheets/2N/2N3904.pdf" H 4850 2950 50  0001 L CNN
+F 4 "C20526" H 4850 2950 50  0001 C CNN "LCSC"
 	1    4850 2950
 	1    0    0    -1
@@
 F 0 "R1" V 4143 2950 50  0000 C CNN
 F 1 "1K" V 4234 2950 50  0000 C CNN
-F 2 "Resistors_SMD:R_0805" V 4280 2950 50  0001 C CNN
+F 2 "Resistors_SMD:R_0603" V 4280 2950 50  0001 C CNN
 F 3 "~" H 4350 2950 50  0001 C CNN
+F 4 "C21190" V 4350 2950 50  0001 C CNN "LCSC"
 	1    4350 2950
 	0    1    1    0
@@
 F 0 "R4" H 5020 2546 50  0000 L CNN
 F 1 "1K" H 5020 2455 50  0000 L CNN
-F 2 "Resistors_SMD:R_0805" V 4880 2500 50  0001 C CNN
+F 2 "Resistors_SMD:R_0603" V 4880 2500 50  0001 C CNN
 F 3 "~" H 4950 2500 50  0001 C CNN
+F 4 "C21190" H 4950 2500 50  0001 C CNN "LCSC"
 	1    4950 2500
 	1    0    0    -1
@@
 F 0 "C1" H 2915 3246 50  0000 L CNN
 F 1 "100nF" H 2915 3155 50  0000 L CNN
-F 2 "Capacitors_SMD:C_0805" H 2838 3050 50  0001 C CNN
+F 2 "Capacitors_SMD:C_0603" H 2838 3050 50  0001 C CNN
 F 3 "~" H 2800 3200 50  0001 C CNN
+F 4 "C14663" H 2800 3200 50  0001 C CNN "LCSC"
 	1    2800 3200
 	1    0    0    -1
@@
 P 5650 2700
 F 0 "Q2" H 5855 2746 50  0000 L CNN
-F 1 "IRLR7821PBF" H 5855 2655 50  0000 L CNN
-F 2 "TO_SOT_Packages_SMD:TO-252-3_TabPin4" H 5900 2625 50  0001 L CIN
-F 3 "http://www.infineon.com/dgdl/irlb8721pbf.pdf?fileId=5546d462533600a40153566056732591" H 5650 2700 50  0001 L CNN
+F 1 "AOD4184A" H 5855 2655 50  0000 L CNN
+F 2 "TO_SOT_Packages_SMD:TO-252-2" H 5900 2625 50  0001 L CIN
+F 3 "https://datasheet.lcsc.com/szlcsc/Alpha-Omega-Semicon-AOS-AOD4184A_C99124.pdf" H 5650 2700 50  0001 L CNN
+F 4 "C99124" H 4850 2950 50  0001 C CNN "LCSC"
 	1    5650 2700
 	1    0    0    -1
@@
 F 2 "Resistors_SMD:R_0603" V 2730 2900 50  0001 C CNN
 F 3 "~" H 2800 2900 50  0001 C CNN
+F 4 "C22775" H 2800 2900 50  0001 C CNN "LCSC"
 	1    2800 2900
 	1    0    0    -1
@@
 F 2 "Resistors_SMD:R_0603" V 2980 2900 50  0001 C CNN
 F 3 "~" H 3050 2900 50  0001 C CNN
+F 4 "C13167" H 3050 2900 50  0001 C CNN "LCSC"
 	1    3050 2900
 	1    0    0    -1
@@
 F 2 "TO_SOT_Packages_SMD:SOT-23" H 5050 3925 50  0001 L CIN
 F 3 "https://www.fairchildsemi.com/datasheets/2N/2N3904.pdf" H 4850 4000 50  0001 L CNN
+F 4 "C20526" H 4850 2950 50  0001 C CNN "LCSC"
 	1    4850 4000
 	1    0    0    -1
@@
 F 0 "R2" V 4143 4000 50  0000 C CNN
 F 1 "1K" V 4234 4000 50  0000 C CNN
-F 2 "Resistors_SMD:R_0805" V 4280 4000 50  0001 C CNN
+F 2 "Resistors_SMD:R_0603" V 4280 4000 50  0001 C CNN
 F 3 "~" H 4350 4000 50  0001 C CNN
+F 4 "C21190" V 4350 4000 50  0001 C CNN "LCSC"
 	1    4350 4000
 	0    1    1    0
@@
 F 0 "R5" H 5020 3596 50  0000 L CNN
 F 1 "1K" H 5020 3505 50  0000 L CNN
-F 2 "Resistors_SMD:R_0805" V 4880 3550 50  0001 C CNN
+F 2 "Resistors_SMD:R_0603" V 4880 3550 50  0001 C CNN
 F 3 "~" H 4950 3550 50  0001 C CNN
+F 4 "C21190" H 4950 3550 50  0001 C CNN "LCSC"
 	1    4950 3550
 	1    0    0    -1
@@
 P 5650 3750
 F 0 "Q5" H 5855 3796 50  0000 L CNN
-F 1 "IRLR7821PBF" H 5855 3705 50  0000 L CNN
-F 2 "TO_SOT_Packages_SMD:TO-252-3_TabPin4" H 5900 3675 50  0001 L CIN
-F 3 "http://www.infineon.com/dgdl/irlb8721pbf.pdf?fileId=5546d462533600a40153566056732591" H 5650 3750 50  0001 L CNN
+F 1 "AOD4184A" H 5855 3705 50  0000 L CNN
+F 2 "TO_SOT_Packages_SMD:TO-252-2" H 5900 3675 50  0001 L CIN
+F 3 "https://datasheet.lcsc.com/szlcsc/Alpha-Omega-Semicon-AOS-AOD4184A_C99124.pdf" H 5650 3750 50  0001 L CNN
+F 4 "C99124" H 5650 3750 50  0001 C CNN "LCSC"
 	1    5650 3750
 	1    0    0    -1
@@
 F 2 "TO_SOT_Packages_SMD:SOT-23" H 5100 4975 50  0001 L CIN
 F 3 "https://www.fairchildsemi.com/datasheets/2N/2N3904.pdf" H 4900 5050 50  0001 L CNN
+F 4 "C20526" H 4900 5050 50  0001 C CNN "LCSC"
 	1    4900 5050
 	1    0    0    -1
@@
 F 0 "R3" V 4193 5050 50  0000 C CNN
 F 1 "1K" V 4284 5050 50  0000 C CNN
-F 2 "Resistors_SMD:R_0805" V 4330 5050 50  0001 C CNN
+F 2 "Resistors_SMD:R_0603" V 4330 5050 50  0001 C CNN
 F 3 "~" H 4400 5050 50  0001 C CNN
+F 4 "C21190" V 4400 5050 50  0001 C CNN "LCSC"
 	1    4400 5050
 	0    1    1    0
@@
 F 0 "R6" H 5070 4646 50  0000 L CNN
 F 1 "1K" H 5070 4555 50  0000 L CNN
-F 2 "Resistors_SMD:R_0805" V 4930 4600 50  0001 C CNN
+F 2 "Resistors_SMD:R_0603" V 4930 4600 50  0001 C CNN
 F 3 "~" H 5000 4600 50  0001 C CNN
+F 4 "C21190" H 5000 4600 50  0001 C CNN "LCSC"
 	1    5000 4600
 	1    0    0    -1
@@
 P 5700 4800
 F 0 "Q6" H 5905 4846 50  0000 L CNN
-F 1 "IRLR7821PBF" H 5905 4755 50  0000 L CNN
-F 2 "TO_SOT_Packages_SMD:TO-252-3_TabPin4" H 5950 4725 50  0001 L CIN
-F 3 "http://www.infineon.com/dgdl/irlb8721pbf.pdf?fileId=5546d462533600a40153566056732591" H 5700 4800 50  0001 L CNN
+F 1 "AOD4184A" H 5905 4755 50  0000 L CNN
+F 2 "TO_SOT_Packages_SMD:TO-252-2" H 5950 4725 50  0001 L CIN
+F 3 "https://datasheet.lcsc.com/szlcsc/Alpha-Omega-Semicon-AOS-AOD4184A_C99124.pdf" H 5700 4800 50  0001 L CNN
+F 4 "C99124" H 5700 4800 50  0001 C CNN "LCSC"
 	1    5700 4800
 	1    0    0    -1
@@
 F 2 "WS2811:SOP-8" H 3250 3500 50  0001 C CNN
 F 3 "https://cdn-shop.adafruit.com/datasheets/WS2811.pdf" H 3350 3600 50  0001 C CNN
+F 4 "C114581" H 3550 3350 50  0001 C CNN "LCSC"
 	1    3550 3350
 	1    0    0    -1
@@
 F 2 "Resistors_SMD:R_0603" V 2480 3400 50  0001 C CNN
 F 3 "~" H 2550 3400 50  0001 C CNN
+F 4 "C23140" V 2550 3400 50  0001 C CNN "LCSC"
 	1    2550 3400
 	0    1    1    0
@@
 F 0 "R12" V 4143 2600 50  0000 C CNN
 F 1 "10K" V 4234 2600 50  0000 C CNN
-F 2 "Resistors_SMD:R_0805" V 4280 2600 50  0001 C CNN
+F 2 "Resistors_SMD:R_0603" V 4280 2600 50  0001 C CNN
 F 3 "~" H 4350 2600 50  0001 C CNN
+F 4 "C25804" V 4350 2600 50  0001 C CNN "LCSC"
 	1    4350 2600
 	0    1    1    0
@@
 F 0 "R13" V 4143 3650 50  0000 C CNN
 F 1 "10K" V 4234 3650 50  0000 C CNN
-F 2 "Resistors_SMD:R_0805" V 4280 3650 50  0001 C CNN
+F 2 "Resistors_SMD:R_0603" V 4280 3650 50  0001 C CNN
 F 3 "~" H 4350 3650 50  0001 C CNN
+F 4 "C25804" V 4350 3650 50  0001 C CNN "LCSC"
 	1    4350 3650
 	0    1    1    0
@@
 F 0 "R14" V 4193 4700 50  0000 C CNN
 F 1 "10K" V 4284 4700 50  0000 C CNN
-F 2 "Resistors_SMD:R_0805" V 4330 4700 50  0001 C CNN
+F 2 "Resistors_SMD:R_0603" V 4330 4700 50  0001 C CNN
 F 3 "~" H 4400 4700 50  0001 C CNN
+F 4 "C25804" V 4400 4700 50  0001 C CNN "LCSC"
 	1    4400 4700
 	0    1    1    0
